Commit message: update

File: model/PFR_Arm/PFR_Arm2.urdf (robot description, URDF)
Before this commit: robot PFR_Arm2, 7 links, 6 joints
Links:
- removed link Joint1_L
- removed link Joint1_R
- removed link Joint2_L
- removed link Joint2_R
- removed link Joint3_L
- removed link Joint3_R
- added link joint1_L, mass 0.410933607210843; collision mesh filename=package://PFR_Arm2/meshes/Joint1_L.STL; visual mesh filename=package://PFR_Arm2/meshes/Joint1_L.STL
- added link joint1_R, mass 0.410933607210843; collision mesh filename=package://PFR_Arm2/meshes/Joint1_R.STL; visual mesh filename=package://PFR_Arm2/meshes/Joint1_R.STL
- added link joint2_L, mass 0.374093067317941; collision mesh filename=package://PFR_Arm2/meshes/Joint2_L.STL; visual mesh filename=package://PFR_Arm2/meshes/Joint2_L.STL
- added link joint2_R, mass 0.374093067317941; collision mesh filename=package://PFR_Arm2/meshes/Joint2_R.STL; visual mesh filename=package://PFR_Arm2/meshes/Joint2_R.STL
- added link joint3_L, mass 0.0882871164231278; collision mesh filename=package://PFR_Arm2/meshes/Joint3_L.STL; visual mesh filename=package://PFR_Arm2/meshes/Joint3_L.STL
- added link joint3_R, mass 0.0882871164231278; collision mesh filename=package://PFR_Arm2/meshes/Joint3_R.STL; visual mesh filename=package://PFR_Arm2/meshes/Joint3_R.STL
- link base_link: geometry collision mesh filename=package://PFR_Arm2/meshes/base_link.STL; visual mesh filename=package://PFR_Arm2/meshes/base_link.STL
Joints:
- removed joint Joint1_L
- removed joint Joint1_R
- removed joint Joint2_L
- removed joint Joint2_R
- removed joint Joint3_L
- removed joint Joint3_R
- added joint joint1_L: type revolute, parent base_link, child joint1_L, origin xyz=0 0.18175 0.174 rpy=0 0 0, axis 0 0 1, limit lower=-1.57079632679 upper=1.57079632679 effort=10 velocity=10
- added joint joint1_R: type revolute, parent base_link, child joint1_R, origin xyz=0 -0.18175 0.174 rpy=0 0 0, axis 0 0 1, limit lower=-1.57079632679 upper=1.57079632679 effort=10 velocity=10
- added joint joint2_L: type revolute, parent joint1_L, child joint2_L, origin xyz=0 0.3 0.00950000000000006 rpy=0 0 0, axis 0 0 1, limit lower=-2.61799387799 upper=2.61799387799 effort=10 velocity=10
- added joint joint2_R: type revolute, parent joint1_R, child joint2_R, origin xyz=0 -0.3 0.00950000000000006 rpy=0 0 0, axis 0 0 1, limit lower=-2.61799387799 upper=2.61799387799 effort=10 velocity=10
- added joint joint3_L: type revolute, parent joint2_L, child joint3_L, origin xyz=0 0.3 0.00949999999999965 rpy=0 0 0, axis 0 0 1, limit lower=-1.57079632679 upper=1.57079632679 effort=10 velocity=10
- added joint joint3_R: type revolute, parent joint2_R, child joint3_R, origin xyz=0 -0.3 0.00949999999999965 rpy=0 0 0, axis 0 0 1, limit lower=-1.57079632679 upper=1.57079632679 effort=10 velocity=10

Commit message: update

File: model/PFR_Arm/PFR_Arm2.urdf (robot description, URDF)
Before this commit: robot PFR_Arm2, 7 links, 6 joints
Joints:
- joint joint1_R: axis 0 0 1 -> 0 0 -1
- joint joint2_R: axis 0 0 1 -> 0 0 -1
- joint joint3_R: axis 0 0 1 -> 0 0 -1

File: src/my_dxl_velocity_cpp/urdf/single_xh540_ros2_control.urdf.xacro (robot description, xacro)
@@ -54,6 +54,6 @@
       <plugin>dynamixel_hardware_interface/DynamixelHardware</plugin>
       <param name="port_name">/dev/ttyUSB0</param>
-      <param name="baud_rate">57600</param>
-      <param name="error_timeout_ms">1000</param>
+      <param name="baud_rate">1000000</param>
+      <param name="error_timeout_ms">250</param>
       <param name="dynamixel_model_folder">/param/dxl_model</param>
       <param name="disable_torque_at_init">true</param>

Commit message: add GJ

File: model/PFR_Arm/PFR_Arm2.urdf (robot description, URDF)
Before this commit: robot PFR_Arm2, 7 links, 6 joints
Links:
- link base_link: mass 37.0077126301145 -> 9.4
- link joint1_L: mass 0.410933607210843 -> 0.610933607210843
- link joint1_R: mass 0.410933607210843 -> 0.610933607210843
- link joint2_L: mass 0.374093067317941 -> 0.524093067317941
- link joint2_R: mass 0.374093067317941 -> 0.524093067317941
- link joint3_L: mass 0.0882871164231278 -> 0.2882871164231278
- link joint3_R: mass 0.0882871164231278 -> 0.2882871164231278

Commit message: changes

File: model/PFR_Arm/PFR_Arm2.urdf (robot description, URDF)
Before this commit: robot PFR_Arm2, 7 links, 6 joints
Links:
- added link world
Joints:
- added joint world_to_base: type floating, parent world, child base_link, origin xyz=0 0 0 rpy=0 0 0

File: model/PFR_Arm/urdf/PFR_Arm2.urdf (robot description, URDF)
Before this commit: robot PFR_Arm2, 7 links, 6 joints
Links:
- added link world
Joints:
- added joint world_to_base: type floating, parent world, child base_link, origin xyz=0 0 0 rpy=0 0 0
